File: Gas_Meter/pcb/PCF8583 1v3.sch (EAGLE design)
At the start: 15 parts, among them IC1 PCF8583P, IC2 A1301UA, IC3 A1301UA, IC4 A1301UA

Commit message: Added text for Jumper J2
Other:
- note added: "Jumper J2 legt die TWI Adresse fest Brücke 1 - 2 : 0x50"
Changed lines of the file:
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@@
 <text x="10.16" y="38.1" size="1.016" layer="91">Hall Sensor AH3661UA
 nur 1 mal an passender Stelle einsetzen</text>
+<text x="40.64" y="38.1" size="1.016" layer="91">Jumper J2 legt die TWI Adresse fest
+Brücke 1 - 2 : 0x50</text>
 </plain>
 <instances>
